Commit message: Implemented ball COG detection and fixed robot behavior

File: my_robot/urdf/my_robot.xacro (robot description, xacro)
@@ -39,5 +39,5 @@
     <pose>0 0 0.1 0 0 0</pose>
     <inertial>
-      <mass value="15.0"/>
+      <mass value="5.0"/>
       <origin xyz="0.0 0 0" rpy=" 0 0 0"/>
       <inertia
@@ -71,16 +71,4 @@
       </geometry>
     </visual>
-    <collision name='front_caster_collision'>
-      <origin xyz="0.15 0 -0.05" rpy=" 0 0 0"/>
-      <geometry>
-        <sphere radius="0.0499"/>
-      </geometry>
-    </collision>
-    <visual name='front_caster_visual'>
-      <origin xyz="0.15 0 -0.05" rpy=" 0 0 0"/>
-      <geometry>
-        <sphere radius="0.05"/>
-      </geometry>
-    </visual>
     <collision name='lidar_mount_collision'>
       <origin xyz="0 0 0.04" rpy=" 0 0 0"/>
@@ -98,5 +86,5 @@
   <link name='left_wheel'>
     <inertial>
-      <mass value="2.0"/>
+      <mass value="1.0"/>
       <inertia
           ixx="0.1" ixy="0" ixz="0"
@@ -119,5 +107,5 @@
   <link name='right_wheel'>
     <inertial>
-      <mass value="2.0"/>
+      <mass value="1.0"/>
       <inertia
           ixx="0.1" ixy="0" ixz="0"

Commit message: Improved robot stability, implemented ball reaching stop

File: my_robot/urdf/my_robot.xacro (robot description, xacro)
@@ -39,5 +39,5 @@
     <pose>0 0 0.1 0 0 0</pose>
     <inertial>
-      <mass value="5.0"/>
+      <mass value="10.0"/>
       <origin xyz="0.0 0 0" rpy=" 0 0 0"/>
       <inertia
@@ -60,5 +60,5 @@
     </visual>
     <collision name='back_caster_collision'>
-      <origin xyz="-0.15 0 -0.05" rpy=" 0 0 0"/>
+      <origin xyz="-0.21 0 -0.05" rpy=" 0 0 0"/>
       <geometry>
         <sphere radius="0.0499"/>
@@ -66,5 +66,17 @@
     </collision>
     <visual name='back_caster_visual'>
-      <origin xyz="-0.15 0 -0.05" rpy=" 0 0 0"/>
+      <origin xyz="-0.21 0 -0.05" rpy=" 0 0 0"/>
+      <geometry>
+        <sphere radius="0.05"/>
+      </geometry>
+    </visual>
+    <collision name='front_caster_collision'>
+      <origin xyz="0.21 0 -0.05" rpy=" 0 0 0"/>
+      <geometry>
+        <sphere radius="0.0499"/>
+      </geometry>
+    </collision>
+    <visual name='front_caster_visual'>
+      <origin xyz="0.21 0 -0.05" rpy=" 0 0 0"/>
       <geometry>
         <sphere radius="0.05"/>

Commit message: Adjustem parameters, removed some objects from map, shifted robot wheel hinges

File: my_robot/urdf/my_robot.xacro (robot description, xacro)
@@ -4,10 +4,10 @@
   <link name="robot_footprint"></link>
   <joint name="robot_footprint_joint" type="fixed">
-    <origin xyz="0 0 0" rpy="0 0 0" />
+    <origin xyz="0 0 0.1" rpy="0 0 0" />
     <parent link="robot_footprint"/>
     <child link="chassis" />
   </joint>
   <joint type="continuous" name="left_wheel_hinge">
-    <origin xyz="0.12 0.2 0" rpy="0 0 0"/>
+    <origin xyz="0.0 0.2 0" rpy="0 0 0"/>
     <child link="left_wheel"/>
     <parent link="chassis"/>
@@ -17,5 +17,5 @@
   </joint>
   <joint type="continuous" name="right_wheel_hinge">
-    <origin xyz="0.12 -0.2 0" rpy="0 0 0"/>
+    <origin xyz="0.0 -0.2 0" rpy="0 0 0"/>
     <child link="right_wheel"/>
     <parent link="chassis"/>

Commit message: Added required files

File: my_robot/urdf/my_robot.xacro (robot description, xacro)
@@ -36,4 +36,12 @@
     <axis xyz="0 1 0"/>
   </joint>
+  <joint name="camera_optical_joint" type="fixed">
+    <!--origin xyz="0 0 0" rpy="-1.5707 0 -1.5707"/-->
+    <origin xyz="0.23 0 0.05" rpy="0 0 0"/>
+    <parent link="camera"/>
+    <child link="camera_link_optical"/>
+  </joint>
+  <link name="camera_link_optical">
+  </link>
   <link name='chassis'>
     <pose>0 0 0.1 0 0 0</pose>

Commit message: Fixed camera orientation

File: my_robot/urdf/my_robot.xacro (robot description, xacro)
@@ -38,5 +38,5 @@
   <joint name="camera_optical_joint" type="fixed">
     <!--origin xyz="0 0 0" rpy="-1.5707 0 -1.5707"/-->
-    <origin xyz="0.23 0 0.05" rpy="0 0 0"/>
+    <origin xyz="0.23 0 0.05" rpy="-1.5707 0 -1.5707"/>
     <parent link="camera"/>
     <child link="camera_link_optical"/>
